Commit message: reference papaer control implement and Arm Exp notebook conclusion

File: model_raisim/DRMPC/SaTiZ_3D/urdf/LISM_Arm_plate.urdf (robot description, URDF)
Before this commit: robot LISM_Arm, 11 links, 10 joints
Links:
- removed link prism_link
- added link anothor
- link hand: mass 0.2 -> 0.064; geometry collision box size=0.12 0.12 0.003; visual box size=0.12 0.12 0.003
Joints:
- joint lower_add: axis 0 0 1 -> 0 1 0; child prism_link -> anothor; type prismatic -> revolute
- joint lower_hand_y: axis 0 1 0 -> 1 0 0; origin xyz=0.0, 0.0, -0.02 rpy=0 0 0 -> xyz=0.0, 0.0, 0.0 rpy=0 0 0; parent prism_link -> anothor

File: model_raisim/LISM_1D/urdf/LISM_Arm_sim.urdf (robot description, URDF)
Before this commit: robot LISM_Arm, 11 links, 10 joints
Joints:
- joint plate_arm_r: axis 1 0 0 -> 0 0 1; origin xyz=0.05 0.1 0.7 rpy=0 0 0 -> xyz=0.0 0.0 0.7 rpy=0 0 0; parent cir_plate_r -> arm_plate; type fixed -> revolute
