Commit message: Paper Sim by z_traj and angle_PD control, torque analysis and visulization

File: model_raisim/DRMPC/SaTiZ_3D/urdf/ball2.urdf (robot description, URDF)
Before this commit: robot LISM_Arm, 2 links, 0 joints
Links:
- added link link0
- added link link1
- link ball: geometry collision sphere radius=0.15; visual mesh filename=meshes/ball2.dae scale=0.001 0.001 0.001
Joints:
- added joint worldTolink1: type fixed, parent world, child link0, origin xyz=0.0 0.0 0.0 rpy=0 0 0
- added joint y: type prismatic, parent link0, child link1, origin xyz=0.0 0.0 0.0 rpy=0 0 0, axis 0.0 1.0 0.0
- added joint z: type prismatic, parent link1, child ball, origin xyz=0.0 0.0 0.0 rpy=0 0 0, axis 0.0 0.0 1
