Commit message: add MPC controller on raisim env and visual code

File: model_raisim/DRMPC/SaTiZ/urdf/TIP copy.urdf (robot description, URDF)
Before this commit: robot LISM_Arm, 5 links, 4 joints
Links:
- link link2: geometry visual cylinder length=0.3 radius=0.03
- link link3: geometry visual cylinder length=0.3 radius=0.03
Joints:
- joint l22l3: origin xyz=0.0 0.0 0.8 rpy=0 0 0 -> xyz=0.0 0.0 0.3 rpy=0 0 0
