Commit message: MPC control complete

File: model_raisim/DRMPC/SaTiZ/urdf/TIP_high_inertia.urdf (robot description, URDF)
Before this commit: robot LISM_Arm, 5 links, 4 joints
Links:
- link link1: mass 10.0 -> 0.5; geometry visual cylinder length=0.8 radius=0.03
- link link2: mass 3.8 -> 0.2
- link link3: mass 3.1 -> 0.2; geometry visual cylinder length=0.3 radius=0.03
Joints:
- joint l12l2: origin xyz=0.0 0.0 1.0 rpy=0 0 0 -> xyz=0.0 0.0 0.8 rpy=0 0 0

File: model_raisim/DRMPC/SaTiZ/urdf/TIP_low.urdf (robot description, URDF)
Before this commit: robot LISM_Arm, 5 links, 4 joints
Links:
- link link1: mass 10.0 -> 0.5; geometry visual cylinder length=0.8 radius=0.03
- link link2: mass 3.8 -> 0.2
- link link3: mass 3.1 -> 0.2; geometry visual cylinder length=0.3 radius=0.03
Joints:
- joint l12l2: origin xyz=0.0 0.0 1.0 rpy=0 0 0 -> xyz=0.0 0.0 0.8 rpy=0 0 0

File: model_raisim/DRMPC/SaTiZ/urdf/TIP_params.urdf (robot description, URDF)
Before this commit: robot LISM_Arm, 5 links, 4 joints
Links:
- link link1: mass 0.5 -> {@@body_mass}; geometry visual cylinder length={@@L_body} radius=0.03
- link link2: mass 0.2 -> {@@thigh_mass}; geometry visual cylinder length={@@L_thigh} radius=0.03
- link link3: mass 0.2 -> {@@shank_mass}; geometry visual cylinder length={@@L_shank} radius=0.03
Joints:
- joint l12l2: origin xyz=0.0 0.0 0.8 rpy=0 0 0 -> xyz=0.0 0.0 {@@L_body} rpy=0 0 0
- joint l22l3: origin xyz=0.0 0.0 0.3 rpy=0 0 0 -> xyz=0.0 0.0 {@@L_thigh} rpy=0 0 0
